File: board/board.brd (EAGLE design)
At the start: 101.6 x 25.4 mm, 46 parts, among them IC1 MCP1703CB

Commit message: Finalize board.
Parts:
- removed IC1: MCP1703CB, linear:SOT23
- removed U$4: LMP7718, custom:SO08
- removed U$5: MAX1837, custom:SOT23-6L
- added OPAMP: LMP7718, custom:SO08
- added UART: (no value), SparkFun:1X03
- added VREG1: MAX1837, custom:SOT23-6L
- added VREG2: MCP1703CB, linear:SOT23
- C10, C7, C8, C9: value (none) -> 10uF
- C16: device rcl:C0805 -> rcl:C1206
- R12: value 5k -> 5.1k
- moved C16 15.3 mm to (75.2, 21.6), turned to 180 degrees
- moved L1 14.3 mm to (74.0, 15.6)
- moved D1 14.1 mm to (73.3, 18.7)
- moved C17 13.7 mm to (80.6, 14.9)
- moved C18 13.7 mm to (75.6, 9.21)
- moved PWR 13.7 mm to (80.3, 21.3)
- moved PROG 3.19 mm to (39.1, 21.9)
- moved MOTOR 3.18 mm to (74.9, 4.13)
- moved C3 3.18 mm to (61.0, 17.8)
- moved C4 3.18 mm to (61.0, 20.0)
- moved C5 3.18 mm to (56.8, 17.8)
- moved C6 3.18 mm to (56.8, 20.0)
- moved R1 3.18 mm to (64.1, 19.1)
- moved U$1 3.18 mm to (41.0, 10.5)
- moved U$3 3.18 mm to (67.0, 13.7)
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Connections:
- new net RX: U$1.P$14, UART.2
- new net TX: U$1.P$11, UART.1
- net ADC_L: now also OPAMP.1; no longer U$4.1
- net ADC_R: now also OPAMP.7; no longer U$4.7
- net GND: now also OPAMP.4, UART.3, VREG1.1, VREG1.2, VREG2.1; no longer IC1.1, U$4.4, U$5.1, U$5.2
- net N$1: now also VREG1.3, VREG1.5; no longer U$5.3, U$5.5
- net N$12: now also OPAMP.5; no longer U$4.5
- net N$13: now also VREG1.4; no longer U$5.4
- net N$6: now also OPAMP.3; no longer U$4.3
- net N$7: now also OPAMP.2; no longer U$4.2
- net N$8: now also OPAMP.6; no longer U$4.6
- net V5: now also VREG1.6, VREG2.3; no longer IC1.3, U$5.6
- net VDD: now also OPAMP.8, VREG2.2; no longer IC1.2, U$4.8
Routing:
- net TX: track 0.00 -> 52.7 mm, vias 0 -> 1
- net RX: track 0.00 -> 48.9 mm, vias 0 -> 1
- net VDD: track 192.5 -> 167.0 mm, vias 0 -> 2
- net V5: track 58.8 -> 46.0 mm, vias 3 -> 1
Other:
- board size 101.6 x 25.4 mm -> 95.2 x 25.4 mm
- board text added: "Aaron Fan"
- board text added: "v0.1"
