File: board/board.sch (EAGLE design)
At the start: 46 parts, among them IC1 MCP1703CB

Commit message: Finalize board.
Parts:
- added UART: (no value), SparkFun:M03PTH
- C10, C7, C8, C9: value (none) -> 10uF
- C16: device rcl:C-USC0805 -> rcl:C-USC1206
- R12: value 5k -> 5.1k
- renumbered IC1 to VREG2, U$4 to OPAMP, U$5 to VREG1
Connections:
- new net RX: U$1.P$14, UART.2
- new net TX: U$1.P$11, UART.1
- net GND: now also UART.3
Changed lines of the file:
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@@
 <part name="R6" library="pot" deviceset="TRIM_US-" device="RJ6S" value="10K"/>
 <part name="R9" library="pot" deviceset="TRIM_US-" device="RJ6S" value="10K"/>
-<part name="C7" library="rcl" deviceset="C-US" device="C1206"/>
-<part name="C8" library="rcl" deviceset="C-US" device="C1206"/>
-<part name="C9" library="rcl" deviceset="C-US" device="C1206"/>
-<part name="C10" library="rcl" deviceset="C-US" device="C1206"/>
+<part name="C7" library="rcl" deviceset="C-US" device="C1206" value="10uF"/>
+<part name="C8" library="rcl" deviceset="C-US" device="C1206" value="10uF"/>
+<part name="C9" library="rcl" deviceset="C-US" device="C1206" value="10uF"/>
+<part name="C10" library="rcl" deviceset="C-US" device="C1206" value="10uF"/>
 <part name="C11" library="rcl" deviceset="C-US" device="C0805" value="1uF"/>
 <part name="PROG" library="SparkFun" deviceset="M05" device="PTH" value=" "/>
@@
 <part name="C14" library="rcl" deviceset="C-US" device="C0805" value="0.1uF"/>
 <part name="C15" library="rcl" deviceset="C-US" device="C0805" value="10uF"/>
-<part name="U$4" library="custom" deviceset="LMP7718" device=""/>
-<part name="IC1" library="linear" deviceset="MCP1703" device="CB"/>
-<part name="U$5" library="custom" deviceset="MAX1837" device=""/>
+<part name="OPAMP" library="custom" deviceset="LMP7718" device=""/>
+<part name="VREG2" library="linear" deviceset="MCP1703" device="CB"/>
+<part name="VREG1" library="custom" deviceset="MAX1837" device=""/>
 <part name="QDECR" library="SparkFun" deviceset="M04" device="POLAR" value=" "/>
 <part name="QDECL" library="SparkFun" deviceset="M04" device="POLAR" value=" "/>
@@
 <part name="PWR" library="SparkFun" deviceset="M02" device="POLAR" value=" "/>
 <part name="MOTOR" library="SparkFun" deviceset="M02" device="POLAR" value=" "/>
-<part name="C16" library="rcl" deviceset="C-US" device="C0805" value="10uF"/>
+<part name="C16" library="rcl" deviceset="C-US" device="C1206" value="10uF"/>
 <part name="C17" library="rcl" deviceset="CPOL-US" device="CT3528" value="150uF"/>
 <part name="L1" library="SparkFun" deviceset="INDUCTOR" device="1007" value="22uH"/>
 <part name="D1" library="SparkFun" deviceset="DIODE" device="SOD" value="d"/>
 <part name="C18" library="rcl" deviceset="C-US" device="C0805" value="10uF"/>
-<part name="R12" library="rcl" deviceset="R-US_" device="R0805" value="5k"/>
+<part name="R12" library="rcl" deviceset="R-US_" device="R0805" value="5.1k"/>
+<part name="UART" library="SparkFun" deviceset="M03" device="PTH"/>
 </parts>
 <sheets>
@@
 <instance part="C14" gate="G$1" x="111.76" y="35.56"/>
 <instance part="C15" gate="G$1" x="68.58" y="-17.78"/>
-<instance part="U$4" gate="G$1" x="259.08" y="45.72" rot="MR0"/>
-<instance part="U$4" gate="G$2" x="261.62" y="-15.24" rot="MR0"/>
-<instance part="IC1" gate="G$1" x="121.92" y="124.46"/>
-<instance part="U$5" gate="G$1" x="50.8" y="119.38"/>
+<instance part="OPAMP" gate="G$1" x="259.08" y="45.72" rot="MR0"/>
+<instance part="OPAMP" gate="G$2" x="261.62" y="-15.24" rot="MR0"/>
+<instance part="VREG2" gate="G$1" x="121.92" y="124.46"/>
+<instance part="VREG1" gate="G$1" x="50.8" y="119.38"/>
 <instance part="QDECR" gate="G$1" x="175.26" y="139.7"/>
 <instance part="QDECL" gate="G$1" x="175.26" y="121.92"/>
@@
 <instance part="C18" gate="G$1" x="137.16" y="121.92"/>
 <instance part="R12" gate="G$1" x="162.56" y="109.22" rot="R90"/>
+<instance part="UART" gate="G$1" x="-33.02" y="73.66"/>
 </instances>
 <busses>
@@
 <wire x1="233.68" y1="66.04" x2="251.46" y2="66.04" width="0.1524" layer="91"/>
 <junction x="251.46" y="66.04"/>
-<pinref part="U$4" gate="G$1" pin="V+"/>
+<pinref part="OPAMP" gate="G$1" pin="V+"/>
 </segment>
 <segment>
@@
 </segment>
 <segment>
-<pinref part="IC1" gate="G$1" pin="VO"/>
+<pinref part="VREG2" gate="G$1" pin="VO"/>
 <wire x1="132.08" y1="124.46" x2="137.16" y2="124.46" width="0.1524" layer="91"/>
 <label x="139.7" y="124.46" size="1.778" layer="95"/>
@@
 </segment>
 <segment>
-<pinref part="IC1" gate="G$1" pin="GND"/>
+<pinref part="VREG2" gate="G$1" pin="GND"/>
 <wire x1="121.92" y1="116.84" x2="121.92" y2="111.76" width="0.1524" layer="91"/>
 <label x="121.92" y="104.14" size="1.778" layer="95"/>
@@
 <wire x1="259.08" y1="35.56" x2="254" y2="35.56" width="0.1524" layer="91"/>
 <label x="254" y="35.56" size="1.778" layer="95"/>
-<pinref part="U$4" gate="G$1" pin="V-"/>
+<pinref part="OPAMP" gate="G$1" pin="V-"/>
 </segment>
 <segment>
@@
 <wire x1="15.24" y1="116.84" x2="15.24" y2="109.22" width="0.1524" layer="91"/>
 <wire x1="15.24" y1="109.22" x2="0" y2="109.22" width="0.1524" layer="91"/>
-<pinref part="U$5" gate="G$1" pin="GND"/>
+<pinref part="VREG1" gate="G$1" pin="GND"/>
 <wire x1="33.02" y1="114.3" x2="30.48" y2="114.3" width="0.1524" layer="91"/>
 <wire x1="30.48" y1="114.3" x2="30.48" y2="109.22" width="0.1524" layer="91"/>
@@
 </segment>
 <segment>
-<pinref part="U$5" gate="G$1" pin="FB"/>
+<pinref part="VREG1" gate="G$1" pin="FB"/>
 <wire x1="68.58" y1="114.3" x2="71.12" y2="114.3" width="0.1524" layer="91"/>
 <wire x1="71.12" y1="114.3" x2="71.12" y2="106.68" width="0.1524" layer="91"/>
@@
 <wire x1="172.72" y1="101.6" x2="162.56" y2="101.6" width="0.1524" layer="91"/>
 <label x="162.56" y="101.6" size="1.778" layer="95"/>
+</segment>
+<segment>
+<pinref part="UART" gate="G$1" pin="3"/>
+<wire x1="-25.4" y1="76.2" x2="-15.24" y2="76.2" width="0.1524" layer="91"/>
+<label x="-17.78" y="76.2" size="1.778" layer="95"/>
 </segment>
 </net>
@@
 <wire x1="276.86" y1="48.26" x2="276.86" y2="50.8" width="0.1524" layer="91"/>
 <junction x="276.86" y="48.26"/>
-<pinref part="U$4" gate="G$1" pin="+IN"/>
+<pinref part="OPAMP" gate="G$1" pin="+IN"/>
 <junction x="266.7" y="48.26"/>
 </segment>
@@
 <wire x1="248.92" y1="27.94" x2="248.92" y2="45.72" width="0.1524" layer="91"/>
 <junction x="248.92" y="45.72"/>
-<pinref part="U$4" gate="G$1" pin="OUT"/>
+<pinref part="OPAMP" gate="G$1" pin="OUT"/>
 </segment>
 <segment>
@@
 <wire x1="248.92" y1="-25.4" x2="248.92" y2="-15.24" width="0.1524" layer="91"/>
 <junction x="248.92" y="-15.24"/>
-<pinref part="U$4" gate="G$2" pin="OUT"/>
+<pinref part="OPAMP" gate="G$2" pin="OUT"/>
 </segment>
 <segment>
@@
 <wire x1="276.86" y1="-12.7" x2="276.86" y2="-10.16" width="0.1524" layer="91"/>
 <junction x="276.86" y="-12.7"/>
-<pinref part="U$4" gate="G$2" pin="+IN"/>
+<pinref part="OPAMP" gate="G$2" pin="+IN"/>
 <junction x="266.7" y="-12.7"/>
 </segment>
@@
 <wire x1="276.86" y1="43.18" x2="276.86" y2="40.64" width="0.1524" layer="91"/>
 <junction x="276.86" y="43.18"/>
-<pinref part="U$4" gate="G$1" pin="-IN"/>
+<pinref part="OPAMP" gate="G$1" pin="-IN"/>
 </segment>
 </net>
@@
 <wire x1="284.48" y1="-17.78" x2="276.86" y2="-17.78" width="0.1524" layer="91"/>
 <junction x="276.86" y="-17.78"/>
-<pinref part="U$4" gate="G$2" pin="-IN"/>
+<pinref part="OPAMP" gate="G$2" pin="-IN"/>
 </segment>
 </net>
@@
 <wire x1="88.9" y1="124.46" x2="93.98" y2="124.46" width="0.1524" layer="91"/>
 <wire x1="93.98" y1="124.46" x2="93.98" y2="121.92" width="0.1524" layer="91"/>
-<pinref part="U$5" gate="G$1" pin="OUT"/>
+<pinref part="VREG1" gate="G$1" pin="OUT"/>
 <wire x1="68.58" y1="119.38" x2="71.12" y2="119.38" width="0.1524" layer="91"/>
 <wire x1="71.12" y1="119.38" x2="71.12" y2="116.84" width="0.1524" layer="91"/>
@@
 <junction x="88.9" y="124.46"/>
 <label x="91.44" y="124.46" size="1.778" layer="95"/>
-<pinref part="IC1" gate="G$1" pin="VI"/>
+<pinref part="VREG2" gate="G$1" pin="VI"/>
 <wire x1="111.76" y1="124.46" x2="93.98" y2="124.46" width="0.1524" layer="91"/>
 <junction x="93.98" y="124.46"/>
@@
 <net name="N$1" class="0">
 <segment>
-<pinref part="U$5" gate="G$1" pin="IN"/>
+<pinref part="VREG1" gate="G$1" pin="IN"/>
 <pinref part="C16" gate="G$1" pin="1"/>
 <wire x1="33.02" y1="124.46" x2="27.94" y2="124.46" width="0.1524" layer="91"/>
@@
 <wire x1="27.94" y1="124.46" x2="27.94" y2="119.38" width="0.1524" layer="91"/>
 <junction x="27.94" y="124.46"/>
-<pinref part="U$5" gate="G$1" pin="!SHDN"/>
+<pinref part="VREG1" gate="G$1" pin="!SHDN"/>
 <wire x1="27.94" y1="119.38" x2="33.02" y2="119.38" width="0.1524" layer="91"/>
 </segment>
@@
 <net name="N$13" class="0">
 <segment>
-<pinref part="U$5" gate="G$1" pin="LX"/>
+<pinref part="VREG1" gate="G$1" pin="LX"/>
 <pinref part="L1" gate="G$1" pin="1"/>
 <wire x1="73.66" y1="124.46" x2="68.58" y2="124.46" width="0.1524" layer="91"/>
@@
 </segment>
 </net>
+<net name="RX" class="0">
+<segment>
+<pinref part="UART" gate="G$1" pin="2"/>
+<wire x1="-25.4" y1="73.66" x2="-15.24" y2="73.66" width="0.1524" layer="91"/>
+<label x="-17.78" y="73.66" size="1.778" layer="95"/>
+</segment>
+<segment>
+<pinref part="U$1" gate="G$1" pin="P$14"/>
+<wire x1="30.48" y1="0" x2="40.64" y2="0" width="0.1524" layer="91"/>
+<label x="30.48" y="0" size="1.778" layer="95"/>
+</segment>
+</net>
+<net name="TX" class="0">
+<segment>
+<pinref part="UART" gate="G$1" pin="1"/>
+<wire x1="-15.24" y1="71.12" x2="-25.4" y2="71.12" width="0.1524" layer="91"/>
+<label x="-17.78" y="71.12" size="1.778" layer="95"/>
+</segment>
+<segment>
+<pinref part="U$1" gate="G$1" pin="P$11"/>
+<wire x1="40.64" y1="7.62" x2="30.48" y2="7.62" width="0.1524" layer="91"/>
+<label x="30.48" y="7.62" size="1.778" layer="95"/>
+</segment>
+</net>
